Commit message: convert visual stl meshes to dae

File: abb_irb1600_support/urdf/irb1600_6_12_macro.xacro (robot description, xacro)
@@ -7,5 +7,5 @@
       <origin xyz="0 0 0" rpy="0 0 0"/>
       <geometry>
-        <mesh filename="package://abb_irb1600_support/meshes/irb1600_6_12/visual/base_link.stl"/>
+        <mesh filename="package://abb_irb1600_support/meshes/irb1600_6_12/visual/base_link.dae"/>
       </geometry>
       <material name="abb_orange">
@@ -26,5 +26,5 @@
       <origin xyz="0 0 0" rpy="0 0 0"/>
       <geometry>
-        <mesh filename="package://abb_irb1600_support/meshes/irb1600_6_12/visual/link_1.stl"/>
+        <mesh filename="package://abb_irb1600_support/meshes/irb1600_6_12/visual/link_1.dae"/>
       </geometry>
       <material name="abb_orange"/>
@@ -42,5 +42,5 @@
       <origin xyz="0 0 0" rpy="0 0 0"/>
       <geometry>
-        <mesh filename="package://abb_irb1600_support/meshes/irb1600_6_12/visual/link_2.stl"/>
+        <mesh filename="package://abb_irb1600_support/meshes/irb1600_6_12/visual/link_2.dae"/>
       </geometry>
       <material name="abb_orange"/>
@@ -58,5 +58,5 @@
       <origin xyz="0 0 0" rpy="0 0 0"/>
       <geometry>
-        <mesh filename="package://abb_irb1600_support/meshes/irb1600_6_12/visual/link_3.stl"/>
+        <mesh filename="package://abb_irb1600_support/meshes/irb1600_6_12/visual/link_3.dae"/>
       </geometry>
       <material name="abb_orange"/>
@@ -74,5 +74,5 @@
       <origin xyz="0 0 0" rpy="0 0 0"/>
       <geometry>
-        <mesh filename="package://abb_irb1600_support/meshes/irb1600_6_12/visual/link_4.stl"/>
+        <mesh filename="package://abb_irb1600_support/meshes/irb1600_6_12/visual/link_4.dae"/>
       </geometry>
       <material name="abb_orange"/>
@@ -90,5 +90,5 @@
       <origin xyz="0 0 0" rpy="0 0 0"/>
       <geometry>
-        <mesh filename="package://abb_irb1600_support/meshes/irb1600_6_12/visual/link_5.stl"/>
+        <mesh filename="package://abb_irb1600_support/meshes/irb1600_6_12/visual/link_5.dae"/>
       </geometry>
       <material name="abb_orange"/>
@@ -106,5 +106,5 @@
       <origin xyz="0 0 0" rpy="0 0 0"/>
       <geometry>
-        <mesh filename="package://abb_irb1600_support/meshes/irb1600_6_12/visual/link_6.stl"/>
+        <mesh filename="package://abb_irb1600_support/meshes/irb1600_6_12/visual/link_6.dae"/>
       </geometry>
       <material name="abb_orange"/>
